File: Ctrl_part.sch (KiCad schematic (older format))
At the start: 59 parts, among them J10 JoystickSwitch, J11 JoystickSwitch, J9 SWD(PLS5), Q13 2N5551S, SW1 SW_Rst, U12 SN74LVC1G08DBVR, U5 AP3216C, U6 STM32G030K6Tx, U7 SSD1306, Y2 CSTCE8M

Commit message: Завершена трассировка печатной платы. Исправлены ошибки в схема.
Parts:
- D4: renamed from D5; footprint LED_THT:LED_D1.8mm_W1.8mm_H2.4mm_Horizontal_O1.27mm_Z1.6mm -> LED_SMD:LED_0603_1608Metric
- J10: footprint Connector_PinSocket_1.27mm:PinSocket_2x03_P1.27mm_Horizontal -> Modules:JoystickSwitch; symbol Connector_Generic:Conn_02x03_Odd_Even -> Modules:JoystickSwitch
- J11: footprint Connector_PinSocket_1.27mm:PinSocket_2x03_P1.27mm_Horizontal -> Modules:EC11_SMD; symbol Connector_Generic:Conn_02x03_Odd_Even -> Modules:EC11-1098
- J9: footprint Connector_PinSocket_1.27mm:PinSocket_1x05_P1.27mm_Vertical -> Connector_PinSocket_1.27mm:PinSocket_1x05_P1.27mm_Vertical_SMD_Pin1Left
- U8: renamed from U7; footprint Modules:SSD1306_I2C -> Modules:SSD1306_2_I2C
- renumbered C13 to C15, C11 to C16, C12 to C17, C16 to C18, C17 to C19, C14 to C20, C35 to C21, C18 to C22, C15 to C23, C19 to C24, C20 to C25, C21 to C26, C22 to C27, C23 to C28, C36 to C29, C24 to C30, C25 to C31, C26 to C32, Q13 to Q16, R36 to R37, R37 to R38, R38 to R39, R34 to R40, R35 to R41, R53 to R42, R54 to R43, R40 to R44, R41 to R45, R42 to R46, R43 to R47, R44 to R48, R45 to R49, R46 to R50, R47 to R51, R48 to R52, R49 to R53, R50 to R54, R51 to R55, R52 to R56, R55 to R57, R56 to R58, R57 to R59, R58 to R60, R59 to R61, R60 to R62, R61 to R63, R62 to R64, R63 to R65, U6 to U10, U12 to U11, U5 to U9
Connections:
- net +3V3: now also C29.1, U11.5 (VCC)
- net EC11_A: now also J11.A; no longer J11.1 (Pin_1)
- net EC11_B: now also J11.B; no longer J11.3 (Pin_3)
- net EC11_E: now also J11.E; no longer J11.5 (Pin_5)
- net GND1: now also C15.2, C16.2, C17.2, C18.1, C20.2, C21.1, C23.2, C24.2, C25.2, C26.2, C27.2, C28.2, C29.2, C30.2, C31.2, C32.2, D4.1 (K), J10.1, J11.C, J11.D, J9.3 (Pin_3), JP2.2 (B), Q16.2 (E), R43.2, R61.1, R63.1, R65.1, SW1.1, U10.5 (VSS/VSSA), U11.3 (GND), U9.3 (GND), Y2.2
- net +5VP renamed +5P
- removed net GND: C15.2, C16.2, C17.2, C18.1, C20.2, C21.1, C23.2, C24.2, C25.2, C26.2, C27.2, C28.2, C30.2, C31.2, C32.2, D4.1 (K), J10.1 (Pin_1), J11.2 (Pin_2), J11.4 (Pin_4), J11.6 (Pin_6), J9.3 (Pin_3), JP2.2 (B), Q16.2 (E), R43.2, R61.1, R63.1, R65.1, SW1.1, U10.5 (VSS/VSSA), U9.3 (GND), Y2.2
Other:
- moved on the sheet: C15, C18, C19, C21, C22, C24, C25, C26, C27, C28, C29, C30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
